File: hardware/hat.kicad_pcb (KiCad board)
At the start: 4 copper layers, 65 x 56 mm, 18 parts, among them J3 40HAT, J6 CONN_02X02, J9 CONN_01X02, Q1 DMG2305UX, Q2 DMMT5401, U2 CAT24C32

Commit message: update an test GH webhook
Parts:
- added J1: Barrel_Jack, Connector_BarrelJack:BarrelJack_Horizontal, F.Cu at (93.6, 100.3)
- added J2: Screw_Terminal_01x02, TerminalBlock_4Ucon:TerminalBlock_4Ucon_1x02_P3.50mm_Horizontal, F.Cu at (128.3, 111.8)
Connections:
- J3 pad 10: (no net) -> Net-(J3-Pad10)
- J3 pad 11: (no net) -> Net-(J3-Pad11)
- J3 pad 12: (no net) -> Net-(J3-Pad12)
- J3 pad 13: (no net) -> Net-(J3-Pad13)
- J3 pad 15: (no net) -> Net-(J3-Pad15)
- J3 pad 16: (no net) -> Net-(J3-Pad16)
- J3 pad 17: (no net) -> Net-(J3-Pad17)
- J3 pad 18: (no net) -> Net-(J3-Pad18)
- J3 pad 19: (no net) -> Net-(J3-Pad19)
- J3 pad 21: (no net) -> Net-(J3-Pad21)
- J3 pad 22: (no net) -> Net-(J3-Pad22)
- J3 pad 23: (no net) -> Net-(J3-Pad23)
- J3 pad 24: (no net) -> Net-(J3-Pad24)
- J3 pad 26: (no net) -> Net-(J3-Pad26)
- J3 pad 29: (no net) -> Net-(J3-Pad29)
- J3 pad 3: (no net) -> Net-(J3-Pad3)
- J3 pad 31: (no net) -> Net-(J3-Pad31)
- J3 pad 32: (no net) -> Net-(J3-Pad32)
- J3 pad 33: (no net) -> Net-(J3-Pad33)
- J3 pad 35: (no net) -> Net-(J3-Pad35)
- J3 pad 36: (no net) -> Net-(J3-Pad36)
- J3 pad 37: (no net) -> Net-(J3-Pad37)
- J3 pad 38: (no net) -> Net-(J3-Pad38)
- J3 pad 40: (no net) -> Net-(J3-Pad40)
- J3 pad 5: (no net) -> Net-(J3-Pad5)
- J3 pad 7: (no net) -> Net-(J3-Pad7)
- J3 pad 8: (no net) -> Net-(J3-Pad8)
